File: compute_module.kicad_pcb (KiCad board)
At the start: 4 copper layers, 93.2 x 51.6 mm, 42 parts, among them J1 2001-1-2-21-00-BK, P1 POWER, P2 HOST, P3 CAM1, Q1 2N7002P.215, Q2 DMP3056L-7, Q3 2N7002P.215, U1 REG1117-3.3, U2 REG1117A-2.5, U3 REG1117A-1.8

Commit message: More via stitching
Routing:
- net GND: track 360.6 -> 483.3 mm, vias 57 -> 76
Changed lines of the file:
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@@
     (thickness 1.6)
     (drawings 4)
-    (tracks 758)
+    (tracks 813)
     (zones 0)
     (modules 42)
@@
   (segment (start 152.8 86.6) (end 152.2 86) (width 0.35) (layer B.Cu) (net 1))
   (segment (start 152.2 86) (end 152.15 86) (width 0.35) (layer B.Cu) (net 1))
+  (segment (start 94.55 88.1) (end 93.3 88.1) (width 0.2) (layer F.Cu) (net 2) (status 400000))
+  (via (at 91.8 86.6) (size 0.45) (drill 0.3) (layers F.Cu B.Cu) (net 2))
+  (segment (start 93.3 88.1) (end 91.8 86.6) (width 0.2) (layer F.Cu) (net 2))
+  (segment (start 103.55 88.1) (end 103.55 86.05) (width 0.2) (layer F.Cu) (net 2) (status 400000))
+  (via (at 104.8 84.8) (size 0.45) (drill 0.3) (layers F.Cu B.Cu) (net 2))
+  (segment (start 103.55 86.05) (end 104.8 84.8) (width 0.2) (layer F.Cu) (net 2))
+  (segment (start 103.85 79.900001) (end 103.85 81.35) (width 0.2) (layer F.Cu) (net 2) (status 400000))
+  (via (at 103.2 82) (size 0.45) (drill 0.3) (layers F.Cu B.Cu) (net 2))
+  (segment (start 103.85 81.35) (end 103.2 82) (width 0.2) (layer F.Cu) (net 2))
+  (segment (start 116.45 79.900001) (end 116.45 82.15) (width 0.2) (layer F.Cu) (net 2) (status 400000))
+  (via (at 115.4 83.2) (size 0.45) (drill 0.3) (layers F.Cu B.Cu) (net 2))
+  (segment (start 116.45 82.15) (end 115.4 83.2) (width 0.2) (layer F.Cu) (net 2))
+  (segment (start 152.45 79.900001) (end 152.45 61.75) (width 0.2) (layer F.Cu) (net 2) (status 400000))
+  (via (at 155.2 59) (size 0.45) (drill 0.3) (layers F.Cu B.Cu) (net 2))
+  (segment (start 152.45 61.75) (end 155.2 59) (width 0.2) (layer F.Cu) (net 2))
+  (segment (start 117.95 96.76) (end 117.95 95.35) (width 0.2) (layer F.Cu) (net 2) (status C00000))
+  (segment (start 117.95 95.35) (end 116.6 94) (width 0.2) (layer F.Cu) (net 2) (status 400000))
+  (via (at 116.6 94) (size 0.45) (drill 0.3) (layers F.Cu B.Cu) (net 2))
+  (segment (start 170.37 99.16) (end 172.64 99.16) (width 0.2) (layer F.Cu) (net 2) (status 400000))
+  (via (at 176.4 95.4) (size 0.45) (drill 0.3) (layers F.Cu B.Cu) (net 2))
+  (segment (start 172.64 99.16) (end 176.4 95.4) (width 0.2) (layer F.Cu) (net 2))
+  (segment (start 178.4 81.725) (end 178.4 81.6) (width 0.2) (layer F.Cu) (net 2) (status C00000))
+  (segment (start 178.4 81.6) (end 176 79.2) (width 0.2) (layer F.Cu) (net 2) (status 400000))
+  (via (at 176 79.2) (size 0.45) (drill 0.3) (layers F.Cu B.Cu) (net 2))
+  (segment (start 171.525 65) (end 171.525 66.125) (width 0.2) (layer F.Cu) (net 2) (status C00000))
+  (segment (start 171.525 66.125) (end 173.2 67.8) (width 0.2) (layer F.Cu) (net 2) (status 400000))
+  (via (at 173.2 67.8) (size 0.45) (drill 0.3) (layers F.Cu B.Cu) (net 2))
+  (segment (start 172.35 61.3) (end 172.35 62.35) (width 0.2) (layer F.Cu) (net 2) (status 400000))
+  (via (at 173.6 63.6) (size 0.45) (drill 0.3) (layers F.Cu B.Cu) (net 2))
+  (segment (start 172.35 62.35) (end 173.6 63.6) (width 0.2) (layer F.Cu) (net 2))
+  (segment (start 178 62.325) (end 178 60.4) (width 0.2) (layer F.Cu) (net 2) (status 400000))
+  (via (at 179 59.4) (size 0.45) (drill 0.3) (layers F.Cu B.Cu) (net 2))
+  (segment (start 178 60.4) (end 179 59.4) (width 0.2) (layer F.Cu) (net 2))
+  (segment (start 154.25 79.900001) (end 154.25 77.95) (width 0.2) (layer F.Cu) (net 2) (status 400000))
+  (via (at 156.4 75.8) (size 0.45) (drill 0.3) (layers F.Cu B.Cu) (net 2))
+  (segment (start 154.25 77.95) (end 156.4 75.8) (width 0.2) (layer F.Cu) (net 2))
+  (segment (start 134.45 79.900001) (end 134.45 61.25) (width 0.2) (layer F.Cu) (net 2) (status 400000))
+  (via (at 133.6 60.4) (size 0.45) (drill 0.3) (layers F.Cu B.Cu) (net 2))
+  (segment (start 134.45 61.25) (end 133.6 60.4) (width 0.2) (layer F.Cu) (net 2))
+  (segment (start 130.85 79.900001) (end 130.85 73.45) (width 0.2) (layer F.Cu) (net 2) (status 400000))
+  (via (at 128.6 71.2) (size 0.45) (drill 0.3) (layers F.Cu B.Cu) (net 2))
+  (segment (start 130.85 73.45) (end 128.6 71.2) (width 0.2) (layer F.Cu) (net 2))
+  (segment (start 118.25 79.900001) (end 118.25 66.95) (width 0.2) (layer F.Cu) (net 2) (status 400000))
+  (via (at 121 64.2) (size 0.45) (drill 0.3) (layers F.Cu B.Cu) (net 2))
+  (segment (start 118.25 66.95) (end 121 64.2) (width 0.2) (layer F.Cu) (net 2))
+  (segment (start 112.85 79.900001) (end 112.85 77.05) (width 0.2) (layer F.Cu) (net 2) (status 400000))
+  (via (at 111 75.2) (size 0.45) (drill 0.3) (layers F.Cu B.Cu) (net 2))
+  (segment (start 112.85 77.05) (end 111 75.2) (width 0.2) (layer F.Cu) (net 2))
+  (segment (start 112.55 88.1) (end 112.55 89.65) (width 0.2) (layer F.Cu) (net 2) (status 400000))
+  (via (at 108 90.4) (size 0.45) (drill 0.3) (layers F.Cu B.Cu) (net 2))
+  (segment (start 111.8 90.4) (end 108 90.4) (width 0.2) (layer B.Cu) (net 2))
+  (segment (start 112 90.2) (end 111.8 90.4) (width 0.2) (layer B.Cu) (net 2))
+  (via (at 112 90.2) (size 0.45) (drill 0.3) (layers F.Cu B.Cu) (net 2))
+  (segment (start 112.55 89.65) (end 112 90.2) (width 0.2) (layer F.Cu) (net 2))
+  (segment (start 121.7 96) (end 121.7 94.5) (width 0.3) (layer F.Cu) (net 2))
+  (via (at 121.2 94) (size 0.45) (drill 0.3) (layers F.Cu B.Cu) (net 2))
+  (segment (start 121.7 94.5) (end 121.2 94) (width 0.3) (layer F.Cu) (net 2))
   (segment (start 119.75 88.1) (end 119.75 89.75) (width 0.2) (layer F.Cu) (net 2))
   (via (at 120 90) (size 0.45) (drill 0.3) (layers F.Cu B.Cu) (net 2))
@@
   (via (at 125.2 98) (size 0.45) (drill 0.3) (layers F.Cu B.Cu) (net 2))
   (segment (start 124.7 97.5) (end 125.2 98) (width 0.3) (layer F.Cu) (net 2))
-  (segment (start 121.7 96) (end 121.7 94.3) (width 0.3) (layer F.Cu) (net 2))
-  (segment (start 121.7 94.3) (end 121.4 94) (width 0.3) (layer F.Cu) (net 2))
   (segment (start 129.2 96) (end 129.2 97.8) (width 0.3) (layer F.Cu) (net 2))
   (via (at 129.6 98.2) (size 0.45) (drill 0.3) (layers F.Cu B.Cu) (net 2))

Commit message: Removed 2.5V regulator and changed bottom ground plane clearence
Parts:
- removed C12, C13: 10uF, Capacitors_Tantalum_SMD:CP_Tantalum_Case-C_EIA-6032-28_Reflow
- removed U2: REG1117A-2.5, TO_SOT_Packages_SMD:SOT-223-3_TabPin2
- added REF**: MountingHole_2.7mm_M2.5_ISO14580, Mounting_Holes:MountingHole_2.7mm_M2.5_ISO14580, F.Cu at (89.8, 104.2)
- added REF**: MountingHole_2.7mm_M2.5_ISO14580, Mounting_Holes:MountingHole_2.7mm_M2.5_ISO14580, F.Cu at (178.6, 104.2)
- added REF**: MountingHole_2.7mm_M2.5_ISO14580, Mounting_Holes:MountingHole_2.7mm_M2.5_ISO14580, F.Cu at (178.6, 57.0)
- added REF**: MountingHole_2.7mm_M2.5_ISO14580, Mounting_Holes:MountingHole_2.7mm_M2.5_ISO14580, F.Cu at (89.8, 57.0)
- moved C14 5.60 mm to (178.0, 65.4)
- moved C9 5.60 mm to (164.6, 76.4)
- moved F1 5.60 mm to (172.0, 76.4)
- moved Q2 5.60 mm to (168.3, 76.4)
- moved C15 5.60 mm to (169.0, 70.6)
- moved P1 5.60 mm to (176.6, 74.8)
- moved U3 5.60 mm to (169.2, 64.6)
Connections:
- C3 pad 1: +2V5 -> +3V3
- C4 pad 1: +2V5 -> +3V3
- D4 pad 2: Net-(C17-Pad1) -> +3V3
- MD1 pad 189: +2V5 -> +3V3
- MD1 pad 190: +2V5 -> +3V3
Routing:
- net GND: track 483.3 -> 559.4 mm, vias 76 -> 86
- net +2V5: track 47.8 -> 0.00 mm, vias 2 -> 0
- net +3V3: track 154.4 -> 184.4 mm, vias 7 -> 10
- net +5V: track 168.0 -> 139.7 mm, vias 6 -> 7
- net +1V8: track 110.5 -> 88.6 mm
- net Net-(C17-Pad1): track 26.6 -> 28.7 mm
