File: power.sch (KiCad schematic (older format))
At the start: 10 parts, among them P1 POWER, Q2 DMP3056L-7, U1 REG1117-3.3, U3 REG1117A-1.8

Commit message: Added datasheet links to BOM
Changed lines of the file:
@@
 F 0 "U1" H 4000 1750 50  0000 C CNN
 F 1 "REG1117-3.3" H 4000 1700 50  0000 C CNN
-F 2 "TO_SOT_Packages_SMD:SOT-223-3_TabPin2" H 4000 1600 50  0000 C CNN
-F 3 "" H 4000 1500 50  0000 C CNN
+F 2 "TO_SOT_Packages_SMD:SOT-223-3_TabPin2" H 4000 1600 50  0001 C CNN
+F 3 "http://www.ti.com/lit/ds/symlink/reg1117.pdf" H 4000 1500 50  0001 C CNN
 	1    4000 1500
 	1    0    0    -1
@@
 F 0 "U3" H 6050 1750 50  0000 C CNN
 F 1 "REG1117A-1.8" H 6050 1700 50  0000 C CNN
-F 2 "TO_SOT_Packages_SMD:SOT-223-3_TabPin2" H 6050 1600 50  0000 C CNN
-F 3 "" H 6050 1500 50  0000 C CNN
+F 2 "TO_SOT_Packages_SMD:SOT-223-3_TabPin2" H 6050 1600 50  0001 C CNN
+F 3 "http://www.ti.com/lit/ds/symlink/reg1117a.pdf" H 6050 1500 50  0001 C CNN
 	1    6050 1500
 	1    0    0    -1
@@
 F 1 "POWER" H 1150 1750 50  0000 C CNN
 F 2 "Connectors:USB_Micro-B" V 1100 1450 50  0001 C CNN
-F 3 "" V 1100 1450 50  0000 C CNN
+F 3 "https://www.tme.eu/en/Document/b7989e722b05f5084c507fb3ad8f02cb/MX-105017-0001.pdf" V 1100 1450 50  0001 C CNN
 	1    1150 1550
 	0    -1   1    0
@@
 F 1 "DMP3056L-7" H 2350 1400 50  0000 L CNN
 F 2 "TO_SOT_Packages_SMD:SOT-23" H 2350 1550 50  0001 C CNN
-F 3 "" H 2150 1450 50  0000 C CNN
+F 3 "https://www.tme.eu/en/Document/250d260377fe1e01ee709e3eafa0c268/DMP3056L.pdf" H 2150 1450 50  0001 C CNN
 	1    2150 1450
 	0    -1   -1   0
@@
 F 1 "2A 6V" V 1800 1350 50  0000 C CNN
 F 2 "Polyfuse_Bourns_MF-PSML:Polyfuse_0805" H 1750 1150 50  0001 L CNN
-F 3 "" H 1700 1350 50  0001 C CNN
+F 3 "https://gr.mouser.com/datasheet/2/54/Bourns_MF-PSML-1159396.pdf" H 1700 1350 50  0001 C CNN
 	1    1700 1350
 	0    1    1    0

Commit message: Initial PCB changes to support CAM0+CAM1
Parts:
- P1: symbol USB_OTG -> USB_OTG-RESCUE-compute_module
Changed lines of the file:
@@
 EESchema Schematic File Version 2
+LIBS:compute_module-rescue
 LIBS:power
 LIBS:device
@@
 $EndComp
 $Comp
-L +5V #PWR041
+L +5V #PWR043
 U 1 1 5C11A324
 P 3300 950
-F 0 "#PWR041" H 3300 800 50  0001 C CNN
+F 0 "#PWR043" H 3300 800 50  0001 C CNN
 F 1 "+5V" H 3300 1090 50  0000 C CNN
 F 2 "" H 3300 950 50  0000 C CNN
@@
 $EndComp
 $Comp
-L GND #PWR042
+L GND #PWR044
 U 1 1 5C11A42C
 P 3300 2100
-F 0 "#PWR042" H 3300 1850 50  0001 C CNN
+F 0 "#PWR044" H 3300 1850 50  0001 C CNN
 F 1 "GND" H 3300 1950 50  0000 C CNN
 F 2 "" H 3300 2100 50  0000 C CNN
@@
 $EndComp
 $Comp
-L GND #PWR043
+L GND #PWR045
 U 1 1 5C11A44A
 P 4000 2100
-F 0 "#PWR043" H 4000 1850 50  0001 C CNN
+F 0 "#PWR045" H 4000 1850 50  0001 C CNN
 F 1 "GND" H 4000 1950 50  0000 C CNN
 F 2 "" H 4000 2100 50  0000 C CNN
@@
 $EndComp
 $Comp
-L +3V3 #PWR044
+L +3V3 #PWR046
 U 1 1 5C11A4AA
 P 4700 950
-F 0 "#PWR044" H 4700 800 50  0001 C CNN
+F 0 "#PWR046" H 4700 800 50  0001 C CNN
 F 1 "+3V3" H 4700 1090 50  0000 C CNN
 F 2 "" H 4700 950 50  0000 C CNN
@@
 $EndComp
 $Comp
-L GND #PWR045
+L GND #PWR047
 U 1 1 5C11A787
 P 4700 2100
-F 0 "#PWR045" H 4700 1850 50  0001 C CNN
+F 0 "#PWR047" H 4700 1850 50  0001 C CNN
 F 1 "GND" H 4700 1950 50  0000 C CNN
 F 2 "" H 4700 2100 50  0000 C CNN
@@
 $EndComp
 $Comp
-L +5V #PWR046
+L +5V #PWR048
 U 1 1 5C11A92B
 P 5350 950
-F 0 "#PWR046" H 5350 800 50  0001 C CNN
+F 0 "#PWR048" H 5350 800 50  0001 C CNN
 F 1 "+5V" H 5350 1090 50  0000 C CNN
 F 2 "" H 5350 950 50  0000 C CNN
@@
 $EndComp
 $Comp
-L GND #PWR047
+L GND #PWR049
 U 1 1 5C11A93A
 P 5350 2100
-F 0 "#PWR047" H 5350 1850 50  0001 C CNN
+F 0 "#PWR049" H 5350 1850 50  0001 C CNN
 F 1 "GND" H 5350 1950 50  0000 C CNN
 F 2 "" H 5350 2100 50  0000 C CNN
@@
 $EndComp
 $Comp
-L GND #PWR048
+L GND #PWR050
 U 1 1 5C11A940
 P 6050 2100
-F 0 "#PWR048" H 6050 1850 50  0001 C CNN
+F 0 "#PWR050" H 6050 1850 50  0001 C CNN
 F 1 "GND" H 6050 1950 50  0000 C CNN
 F 2 "" H 6050 2100 50  0000 C CNN
@@
 $EndComp
 $Comp
-L GND #PWR049
+L GND #PWR051
 U 1 1 5C11A954
 P 6750 2100
-F 0 "#PWR049" H 6750 1850 50  0001 C CNN
+F 0 "#PWR051" H 6750 1850 50  0001 C CNN
 F 1 "GND" H 6750 1950 50  0000 C CNN
 F 2 "" H 6750 2100 50  0000 C CNN
@@
 $EndComp
 $Comp
-L +1V8 #PWR050
+L +1V8 #PWR052
 U 1 1 5C11AE43
 P 6750 950
-F 0 "#PWR050" H 6750 800 50  0001 C CNN
+F 0 "#PWR052" H 6750 800 50  0001 C CNN
 F 1 "+1V8" H 6750 1090 50  0000 C CNN
 F 2 "" H 6750 950 50  0000 C CNN
@@
 $EndComp
 $Comp
-L USB_OTG P1
+L USB_OTG-RESCUE-compute_module P1
 U 1 1 5C121D56
 P 1150 1550
@@
 NoConn ~ 1450 1650
 $Comp
-L GND #PWR051
+L GND #PWR053
 U 1 1 5C12209B
 P 1050 2100
-F 0 "#PWR051" H 1050 1850 50  0001 C CNN
+F 0 "#PWR053" H 1050 1850 50  0001 C CNN
 F 1 "GND" H 1050 1950 50  0000 C CNN
 F 2 "" H 1050 2100 50  0000 C CNN
@@
 $EndComp
 $Comp
-L +5V #PWR052
+L +5V #PWR054
 U 1 1 5C122165
 P 2600 950
-F 0 "#PWR052" H 2600 800 50  0001 C CNN
+F 0 "#PWR054" H 2600 800 50  0001 C CNN
 F 1 "+5V" H 2600 1090 50  0000 C CNN
 F 2 "" H 2600 950 50  0000 C CNN
@@
 $EndComp
 $Comp
-L GND #PWR053
+L GND #PWR055
 U 1 1 5C122303
 P 1550 2100
-F 0 "#PWR053" H 1550 1850 50  0001 C CNN
+F 0 "#PWR055" H 1550 1850 50  0001 C CNN
 F 1 "GND" H 1550 1950 50  0000 C CNN
 F 2 "" H 1550 2100 50  0000 C CNN
@@
 $EndComp
 $Comp
-L GND #PWR054
+L GND #PWR056
 U 1 1 5C122AC6
 P 2600 2100
-F 0 "#PWR054" H 2600 1850 50  0001 C CNN
+F 0 "#PWR056" H 2600 1850 50  0001 C CNN
 F 1 "GND" H 2600 1950 50  0000 C CNN
 F 2 "" H 2600 2100 50  0000 C CNN
@@
 	2350 1350 2900 1350
 $Comp
-L GND #PWR055
+L GND #PWR057
 U 1 1 5C124E5D
 P 2150 2100
-F 0 "#PWR055" H 2150 1850 50  0001 C CNN
+F 0 "#PWR057" H 2150 1850 50  0001 C CNN
 F 1 "GND" H 2150 1950 50  0000 C CNN
 F 2 "" H 2150 2100 50  0000 C CNN
@@
 Connection ~ 6750 1450
 $Comp
-L PWR_FLAG #FLG056
+L PWR_FLAG #FLG058
 U 1 1 5C13F037
 P 2900 1000
-F 0 "#FLG056" H 2900 1095 50  0001 C CNN
+F 0 "#FLG058" H 2900 1095 50  0001 C CNN
 F 1 "PWR_FLAG" H 2900 1180 50  0000 C CNN
 F 2 "" H 2900 1000 50  0000 C CNN
@@
 	2900 1350 2900 1000
 $Comp
-L PWR_FLAG #FLG057
+L PWR_FLAG #FLG059
 U 1 1 5C13F5FD
 P 7400 1000
-F 0 "#FLG057" H 7400 1095 50  0001 C CNN
+F 0 "#FLG059" H 7400 1095 50  0001 C CNN
 F 1 "PWR_FLAG" H 7400 1180 50  0000 C CNN
 F 2 "" H 7400 1000 50  0000 C CNN
@@
 $EndComp
 $Comp
-L GND #PWR058
+L GND #PWR060
 U 1 1 5C13F62F
 P 7400 2100
-F 0 "#PWR058" H 7400 1850 50  0001 C CNN
+F 0 "#PWR060" H 7400 1850 50  0001 C CNN
 F 1 "GND" H 7400 1950 50  0000 C CNN
 F 2 "" H 7400 2100 50  0000 C CNN
